File: Electrical/KiCad_templates/Expansion_Card/Expansion_Card.kicad_pcb (KiCad board)
At the start: 2 copper layers, 26 x 30 mm, 11 parts, among them P1 USB_C_Plug_USB2.0, U1 AP2112K-3.3

Commit message: Schematic done, Currently routing
Parts:
- removed C1, C2: 10uF, Capacitor_SMD:C_0805_2012Metric
- removed P1: USB_C_Plug_USB2.0, Expansion_Card:USB_C_Plug_Molex_105444
- removed U1: AP2112K-3.3, Package_TO_SOT_SMD:SOT-23-5
- added USB1: 1054440011, easyeda2kicad:USB-C-SMD_C561769, F.Cu at (140.0, 129.5)
- added USB2: HC-USB3.0-C34-P, easyeda2kicad:USB-3.0-A-SMD_HC-USB3.0-C34-P, F.Cu at (140.7, 149.3)
- R1: footprint Resistor_SMD:R_0603_1608Metric -> Resistor_SMD:R_0603_1608Metric_Pad0.98x0.95mm_HandSolder
- moved R1 4.80 mm to (134.0, 131.3)
Connections:
- R1 pad 1: Net-(P1-PadA5) -> GND
- R1 pad 2: GND -> /CC
Routing:
- net /CC: track 0.00 -> 7.13 mm, vias 0 -> 2
- net (no net): vias 0 -> 2
- added copper zone on B.Cu, net GND
- added copper zone on F.Cu, net GND
Other:
- outline, holes or cut-outs redrawn
- net class Default removed
