File: Electrical/KiCad_templates/Expansion_Card/Expansion_Card.kicad_sch (KiCad schematic)
At the start: 4 parts, among them U1 U261-241N-4BC2SS

Commit message: Updated PCB and Re-Ordered
+ Added Local Libraries to Project
Connections:
- net CC is gone; now on net SBU2: U1.B8 (SBU2), USB1.B8 (SUB2)
- net Vconn is gone; now on net SBU1: U1.A8 (SBU1), USB1.A8 (SUB1)
- net RX1+: now also U1.B11 (RX1+), USB1.B11 (SSRXp1); no longer U1.A2 (TX1+), USB1.A2 (SSTXP1)
- net RX1-: now also U1.B10 (RX1-), USB1.B10 (SSRXn1); no longer U1.A3 (TX1-), USB1.A3 (SSTXn1)
- net RX2+: now also U1.A11 (RX2+), USB1.A11 (SSRXp2); no longer U1.B2 (TX2+), USB1.B2 (SSTXp2)
- net RX2-: now also U1.A10 (RX2-), USB1.A10 (SSRXn2); no longer U1.B3 (TX2-), USB1.B3 (SSTXn2)
- net SBU1: no longer U1.B5 (Vconn), USB1.B5 (CC2)
- net SBU2: no longer U1.A5 (CC), USB1.A5 (CC1)
- net TX1+: now also U1.A2 (TX1+), USB1.A2 (SSTXP1); no longer U1.B11 (RX1+), USB1.B11 (SSRXp1)
- net TX1-: now also U1.A3 (TX1-), USB1.A3 (SSTXn1); no longer U1.B10 (RX1-), USB1.B10 (SSRXn1)
- net TX2+: now also U1.B2 (TX2+), USB1.B2 (SSTXp2); no longer U1.A11 (RX2+), USB1.A11 (SSRXp2)
- net TX2-: now also U1.B3 (TX2-), USB1.B3 (SSTXn2); no longer U1.A10 (RX2-), USB1.A10 (SSRXn2)
- net USB_DN: now also U1.B7 (D-); no longer U1.B6 (D+)
- net USB_DP: now also U1.B6 (D+); no longer U1.B7 (D-)
- new net CC1: U1.A5 (CC), USB1.A5 (CC1)
- new net CC2: U1.B5 (Vconn), USB1.B5 (CC2)
Changed lines of the file:
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@@
 	(wire
 		(pts
-			(xy 142.24 54.61) (xy 138.43 54.61)
+			(xy 143.51 54.61) (xy 138.43 54.61)
 		)
 		(stroke
@@
 	(wire
 		(pts
-			(xy 33.02 53.34) (xy 36.83 53.34)
+			(xy 31.75 53.34) (xy 36.83 53.34)
 		)
 		(stroke
@@
 		)
 	)
+	(label "USB_DN"
+		(at 99.06 57.15 0)
+		(effects
+			(font
+				(size 1.27 1.27)
+			)
+			(justify left bottom)
+		)
+	)
 	(label "TX2+"
 		(at 100.33 69.85 0)
@@
 		)
 	)
-	(label "CC"
-		(at 142.24 54.61 180)
+	(label "CC1"
+		(at 143.51 54.61 180)
 		(effects
 			(font
@@
 		)
 	)
-	(label "Vconn"
+	(label "CC2"
 		(at 99.06 62.23 0)
 		(effects
@@
 		)
 	)
-	(label "USB_DP"
-		(at 99.06 57.15 0)
-		(effects
-			(font
-				(size 1.27 1.27)
-			)
-			(justify left bottom)
-		)
-	)
-	(label "Vconn"
+	(label "CC2"
 		(at 68.58 60.96 180)
 		(effects
@@
 		)
 	)
+	(label "USB_DN"
+		(at 68.58 55.88 180)
+		(effects
+			(font
+				(size 1.27 1.27)
+			)
+			(justify right bottom)
+		)
+	)
 	(label "TX2-"
 		(at 100.33 67.31 0)
@@
 		)
 	)
-	(label "USB_DN"
+	(label "USB_DP"
+		(at 99.06 59.69 0)
+		(effects
+			(font
+				(size 1.27 1.27)
+			)
+			(justify left bottom)
+		)
+	)
+	(label "USB_DP"
 		(at 68.58 58.42 180)
 		(effects
@@
 		)
 	)
-	(label "USB_DN"
-		(at 99.06 59.69 0)
-		(effects
-			(font
-				(size 1.27 1.27)
-			)
-			(justify left bottom)
-		)
-	)
-	(label "USB_DP"
-		(at 68.58 55.88 180)
-		(effects
-			(font
-				(size 1.27 1.27)
-			)
-			(justify right bottom)
-		)
-	)
-	(label "USB_DN"
-		(at 147.32 57.15 180)
-		(effects
-			(font
-				(size 1.27 1.27)
-			)
-			(justify right bottom)
-		)
-	)
-	(label "CC"
-		(at 33.02 53.34 0)
+	(label "CC1"
+		(at 31.75 53.34 0)
 		(effects
 			(font
@@
 	)
 	(label "USB_DP"
+		(at 147.32 57.15 180)
+		(effects
+			(font
+				(size 1.27 1.27)
+			)
+			(justify right bottom)
+		)
+	)
+	(label "USB_DN"
 		(at 147.32 59.69 180)
 		(effects
@@
 		(lib_id "easyeda2kicad:TYPE-C24PQT143")
 		(at 123.19 59.69 0)
+		(mirror y)
 		(unit 1)
 		(body_style 1)
@@
 		(in_pos_files yes)
 		(dnp no)
-		(fields_autoplaced yes)
 		(property "Reference" "USB1"
 			(at 123.19 34.29 0)
@@
 		(lib_id "easyeda2kicad:U261-241N-4BC2SS")
 		(at 48.26 57.15 0)
+		(mirror y)
 		(unit 1)
 		(body_style 1)
@@
 		(in_pos_files yes)
 		(dnp no)
-		(fields_autoplaced yes)
 		(property "Reference" "U1"
-			(at 50.4033 35.56 0)
+			(at 46.1167 35.56 0)
 			(show_name no)
 			(do_not_autoplace no)
@@
 		)
 		(property "Value" "U261-241N-4BC2SS"
-			(at 50.4033 38.1 0)
-			(show_name no)
-			(do_not_autoplace no)
+			(at 46.1167 38.1 0)
+			(show_name no)
+			(do_not_autoplace no)

Commit message: Updated to use local footprint library
Parts:
- U1: footprint easyeda2kicad:USB-C-SMD_XKB_U261-24XN-4BC2SS -> project_library:USB-C-SMD_XKB_U261-24XN-4BC2SS
- USB1: footprint easyeda2kicad:TYPE-C-SMD_C9900025773 -> project_library:TYPE-C-SMD_C9900025773
Changed lines of the file:
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@@
 			)
 		)
-		(property "Footprint" "easyeda2kicad:TYPE-C-SMD_C9900025773"
+		(property "Footprint" "project_library:TYPE-C-SMD_C9900025773"
 			(at 123.19 87.63 0)
 			(hide yes)
@@
 			)
 		)
-		(property "Footprint" "easyeda2kicad:USB-C-SMD_XKB_U261-24XN-4BC2SS"
+		(property "Footprint" "project_library:USB-C-SMD_XKB_U261-24XN-4BC2SS"
 			(at 48.26 83.82 0)
 			(hide yes)
